File: WiFi load switch.kicad_pcb (KiCad board)
At the start: 2 copper layers, 56 x 28 mm, 20 parts, among them J1 Debug connector, J2 max. 24V Input, J3 max. 24V output, Q1 Q_NMOS_GDSD, SW1 SW_Push, U1 ESP-12E, U2 LM2594

Commit message: Completed layout. Need to consider housing.
Parts:
- moved R4 2.90 mm to (126.7, 110.0)
- moved R5 0.12 mm to (126.7, 108.4)
Routing:
- net GND: track 0.00 -> 190.1 mm, vias 5 -> 93
- net +3V3: track 37.1 -> 97.9 mm, vias 4 -> 5
- net Net-(R4-Pad2): track 10.6 -> 13.3 mm
- net LED: track 33.8 -> 33.0 mm
- added copper zone on F.Cu, net +3V3
Other:
- outline, holes or cut-outs redrawn
- board text added: "GND RX TX VDD"
- board text added: "HA4TI 2018.03."

Commit message: Minor changes. Design was sent to PCB manufacturer
Parts:
- moved R5 15.8 mm to (111.5, 112.8), turned to 180 degrees
- moved R4 1.14 mm to (127.6, 109.3), turned to 90 degrees
- turned SW1 to 0 degrees
Connections:
- U1 pad 9: Net-(U1-Pad9) -> GND
Routing:
- net GND: track 190.1 -> 327.4 mm, vias 93 -> 92
- net Net-(R4-Pad2): track 13.3 -> 19.7 mm, vias 0 -> 1
- net +3V3: track 97.9 -> 99.7 mm
Other:
- board text added: "6-24V DC input"
- board text added: "ESP-12E: GPIO0 - Switch input GPIO12 - MOSFET, active high GPIO13 - LED, active low"
- board text added: "FDT459N"
- board text added: "LM2594M"
