File: WiFi load switch.sch (KiCad schematic (older format))
At the start: 20 parts, among them J1 Debug connector, J2 max. 24V Input, J3 max. 24V output, Q1 Q_NMOS_GDSD, SW1 SW_Push, U1 ESP-12E, U2 LM2594

Commit message: Minor changes. Design was sent to PCB manufacturer
Connections:
- net GND: now also U1.9 (GND)
Changed lines of the file:
@@
 Wire Wire Line
 	5550 2400 5750 2400
+$Comp
+L GND #PWR?
+U 1 1 5AB4D950
+P 5000 4650
+F 0 "#PWR?" H 5000 4400 50  0001 C CNN
+F 1 "GND" H 5000 4500 50  0000 C CNN
+F 2 "" H 5000 4650 50  0001 C CNN
+F 3 "" H 5000 4650 50  0001 C CNN
+	1    5000 4650
+	1    0    0    -1
+$EndComp
 $EndSCHEMATC
